File: ZX Spectrum, BUS Expander.kicad_sch (KiCad schematic)
At the start: 15 parts, among them J1 Conn_02x28_Row_Letter_First, J2 Conn_02x28_Row_Letter_First, SW1 SW_Push_Dual

Commit message: Sche + Render
Parts:
- removed R3: 100R, Resistor_SMD:R_1206_3216Metric, symbol Device:R
- removed SW1: SW_Push_Dual, Button_Switch_SMD:SW_Push_1P1T_XKB_TS-1187A, symbol Switch:SW_Push_Dual
Other:
- moved on the sheet: C1, D1, H1, H2, H3, H4, R1, R2, S1
